File: Hardware/Schematics/PowerSocket2.sch (EAGLE design)
At the start: 79 parts, among them IC1 REG1117, IC3 74AC373DW, J1 1X2-3.5MM, J2 1X2-3.5MM, J3 1X2-3.5MM, J4 1X2-3.5MM, J5 1X2-3.5MM, J6 1X2-3.5MM, J7 1X2-3.5MM, J8 1X2-3.5MM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

Commit message: Fixed some issues in the schematic.
Parts:
- added R17: 100K, rcl:R-EU_R0805
Connections:
- net GND: now also IC3A.4D, IC3A.5D, IC3A.6D, IC3A.7D, IC3A.8D, R17.2
- net N$32: now also R17.1

Commit message: Try to save schematic for lower version of eagle.
Parts:
- D3, D5, D6, D7: device diode:1N4004 -> diode@1:1N4004
Changed lines of the file:
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@@
 <part name="GND19" library="supply1" deviceset="GND" device=""/>
 <part name="J3" library="adafruit" deviceset="1X2" device="-3.5MM"/>
-<part name="4.5" library="supply1" library_urn="urn:adsk.eagle:library:371" deviceset="VSS" device=""/>
-<part name="4.1" library="supply1" library_urn="urn:adsk.eagle:library:371" deviceset="VSS" device=""/>
+<part name="4.5" library="supply1@1" deviceset="VSS" device=""/>
+<part name="4.1" library="supply1@1" deviceset="VSS" device=""/>
 <part name="R4" library="rcl" deviceset="R-EU_" device="R0805" value="15K"/>
 <part name="J1" library="adafruit" deviceset="1X2" device="-3.5MM"/>
 <part name="J2" library="adafruit" deviceset="1X2" device="-3.5MM"/>
-<part name="SUPPLY3" library="supply2" library_urn="urn:adsk.eagle:library:372" deviceset="VDD" device=""/>
-<part name="SUPPLY4" library="supply2" library_urn="urn:adsk.eagle:library:372" deviceset="VDD" device=""/>
+<part name="SUPPLY3" library="supply2@1" deviceset="VDD" device=""/>
+<part name="SUPPLY4" library="supply2@1" deviceset="VDD" device=""/>
 <part name="J4" library="adafruit" deviceset="1X2" device="-3.5MM"/>
-<part name="AGND1" library="supply1" library_urn="urn:adsk.eagle:library:371" deviceset="AGND" device=""/>
-<part name="SUPPLY5" library="supply2" library_urn="urn:adsk.eagle:library:372" deviceset="VDD" device=""/>
-<part name="AGND2" library="supply1" library_urn="urn:adsk.eagle:library:371" deviceset="AGND" device=""/>
-<part name="OK1" library="optocoupler" library_urn="urn:adsk.eagle:library:320" deviceset="PC817" device=""/>
-<part name="SUPPLY6" library="supply2" library_urn="urn:adsk.eagle:library:372" deviceset="VDD" device=""/>
+<part name="AGND1" library="supply1@1" deviceset="AGND" device=""/>
+<part name="SUPPLY5" library="supply2@1" deviceset="VDD" device=""/>
+<part name="AGND2" library="supply1@1" deviceset="AGND" device=""/>
+<part name="OK1" library="optocoupler" deviceset="PC817" device=""/>
+<part name="SUPPLY6" library="supply2@1" deviceset="VDD" device=""/>
 <part name="R5" library="rcl" deviceset="R-EU_" device="R0805" value="500"/>
 <part name="SUPPLY7" library="supply2" deviceset="+5V" device=""/>
@@
 <part name="D1" library="diode" deviceset="DIODE-" device="DO-214AC"/>
 <part name="R8" library="rcl" deviceset="R-EU_" device="R0805" value="100K"/>
-<part name="4.2" library="supply1" library_urn="urn:adsk.eagle:library:371" deviceset="VSS" device=""/>
+<part name="4.2" library="supply1@1" deviceset="VSS" device=""/>
 <part name="R9" library="rcl" deviceset="R-EU_" device="R0805" value="15K"/>
 <part name="J5" library="adafruit" deviceset="1X2" device="-3.5MM"/>
 <part name="J6" library="adafruit" deviceset="1X2" device="-3.5MM"/>
-<part name="SUPPLY8" library="supply2" library_urn="urn:adsk.eagle:library:372" deviceset="VDD" device=""/>
-<part name="SUPPLY9" library="supply2" library_urn="urn:adsk.eagle:library:372" deviceset="VDD" device=""/>
-<part name="AGND3" library="supply1" library_urn="urn:adsk.eagle:library:371" deviceset="AGND" device=""/>
-<part name="OK2" library="optocoupler" library_urn="urn:adsk.eagle:library:320" deviceset="PC817" device=""/>
-<part name="SUPPLY10" library="supply2" library_urn="urn:adsk.eagle:library:372" deviceset="VDD" device=""/>
+<part name="SUPPLY8" library="supply2@1" deviceset="VDD" device=""/>
+<part name="SUPPLY9" library="supply2@1" deviceset="VDD" device=""/>
+<part name="AGND3" library="supply1@1" deviceset="AGND" device=""/>
+<part name="OK2" library="optocoupler" deviceset="PC817" device=""/>
+<part name="SUPPLY10" library="supply2@1" deviceset="VDD" device=""/>
 <part name="R10" library="rcl" deviceset="R-EU_" device="R0805" value="500"/>
 <part name="SUPPLY11" library="supply2" deviceset="+5V" device=""/>
@@
 <part name="D2" library="diode" deviceset="DIODE-" device="DO-214AC"/>
 <part name="R12" library="rcl" deviceset="R-EU_" device="R0805" value="100K"/>
-<part name="4.3" library="supply1" library_urn="urn:adsk.eagle:library:371" deviceset="VSS" device=""/>
+<part name="4.3" library="supply1@1" deviceset="VSS" device=""/>
 <part name="R13" library="rcl" deviceset="R-EU_" device="R0805" value="15K"/>
 <part name="J7" library="adafruit" deviceset="1X2" device="-3.5MM"/>
 <part name="J8" library="adafruit" deviceset="1X2" device="-3.5MM"/>
-<part name="SUPPLY12" library="supply2" library_urn="urn:adsk.eagle:library:372" deviceset="VDD" device=""/>
-<part name="SUPPLY13" library="supply2" library_urn="urn:adsk.eagle:library:372" deviceset="VDD" device=""/>
-<part name="AGND4" library="supply1" library_urn="urn:adsk.eagle:library:371" deviceset="AGND" device=""/>
-<part name="OK3" library="optocoupler" library_urn="urn:adsk.eagle:library:320" deviceset="PC817" device=""/>
-<part name="SUPPLY14" library="supply2" library_urn="urn:adsk.eagle:library:372" deviceset="VDD" device=""/>
+<part name="SUPPLY12" library="supply2@1" deviceset="VDD" device=""/>
+<part name="SUPPLY13" library="supply2@1" deviceset="VDD" device=""/>
+<part name="AGND4" library="supply1@1" deviceset="AGND" device=""/>
+<part name="OK3" library="optocoupler" deviceset="PC817" device=""/>
+<part name="SUPPLY14" library="supply2@1" deviceset="VDD" device=""/>
 <part name="R14" library="rcl" deviceset="R-EU_" device="R0805" value="500"/>
 <part name="SUPPLY15" library="supply2" deviceset="+5V" device=""/>
-<part name="IC3" library="74xx-eu" library_urn="urn:adsk.eagle:library:85" deviceset="74*373" device="DW" technology="AC"/>
+<part name="IC3" library="74xx-eu" deviceset="74*373" device="DW" technology="AC"/>
 <part name="GND20" library="supply1" deviceset="GND" device=""/>
-<part name="HCPL-7520" library="avago" library_urn="urn:adsk.eagle:library:107" deviceset="HCPL-7800" device="A"/>
-<part name="SUPPLY16" library="supply2" library_urn="urn:adsk.eagle:library:372" deviceset="VDD" device=""/>
-<part name="AGND5" library="supply1" library_urn="urn:adsk.eagle:library:371" deviceset="AGND" device=""/>
+<part name="HCPL-7520" library="avago" deviceset="HCPL-7800" device="A"/>
+<part name="SUPPLY16" library="supply2@1" deviceset="VDD" device=""/>
+<part name="AGND5" library="supply1@1" deviceset="AGND" device=""/>
 <part name="C11" library="rcl" deviceset="C-EU" device="C1206" value="100nF"/>
 <part name="J9" library="adafruit" deviceset="1X2" device="-3.5MM"/>
-<part name="D3" library="diode" library_urn="urn:adsk.eagle:library:210" deviceset="1N4004" device=""/>
-<part name="D5" library="diode" library_urn="urn:adsk.eagle:library:210" deviceset="1N4004" device=""/>
-<part name="D6" library="diode" library_urn="urn:adsk.eagle:library:210" deviceset="1N4004" device=""/>
-<part name="D7" library="diode" library_urn="urn:adsk.eagle:library:210" deviceset="1N4004" device=""/>
-<part name="R15" library="resistor" library_urn="urn:adsk.eagle:library:348" deviceset="R-EU_" device="0207/10" value="1M"/>
-<part name="R16" library="resistor" library_urn="urn:adsk.eagle:library:348" deviceset="R-EU_" device="0207/10" value="8.2K"/>
+<part name="D3" library="diode@1" deviceset="1N4004" device=""/>
+<part name="D5" library="diode@1" deviceset="1N4004" device=""/>
+<part name="D6" library="diode@1" deviceset="1N4004" device=""/>
+<part name="D7" library="diode@1" deviceset="1N4004" device=""/>
+<part name="R15" library="resistor" deviceset="R-EU_" device="0207/10" value="1M"/>
+<part name="R16" library="resistor" deviceset="R-EU_" device="0207/10" value="8.2K"/>
 <part name="P+6" library="supply1" deviceset="VCC" device=""/>
 <part name="GND21" library="supply1" deviceset="GND" device=""/>
@@
 </schematic>
 </drawing>
-<compatibility>
-<note version="8.2" severity="warning">
-Since Version 8.2, Eagle supports online libraries. The ids
-of those online libraries will not be understood (or retained)
-with this version.
-</note>
-</compatibility>
 </eagle>

Commit message: Return OK in settings.
Connections:
- net FLASH: now also U1.IO0; no longer U1.IO4
Changed lines of the file:
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@@
 </segment>
 <segment>
-<pinref part="U1" gate="G$1" pin="IO4"/>
-<wire x1="30.48" y1="-2.54" x2="53.34" y2="-2.54" width="0.1524" layer="91"/>
-<label x="48.72" y="-2.32" size="1.778" layer="95"/>
+<pinref part="U1" gate="G$1" pin="IO0"/>
+<wire x1="30.48" y1="-5.08" x2="40.64" y2="-5.08" width="0.1524" layer="91"/>
+<label x="33.02" y="-5.08" size="1.778" layer="95"/>
 </segment>
 </net>
